Commit message: add qr_track.cpp

File: mbot_description/urdf/xacro/gazebo/mbot_base.xacro (robot description, xacro)
@@ -146,6 +146,6 @@
         <xacro:wheel prefix="left"  reflect="-1"/>
         <xacro:wheel prefix="right" reflect="1"/>
-        <xacro:caster prefix="front" reflect="-1"/>
-        <xacro:caster prefix="back"  reflect="1"/>
+        <xacro:caster prefix="front" reflect="1"/>
+        <xacro:caster prefix="back"  reflect="-1"/>
         <!-- controller -->
         <gazebo>
@@ -153,5 +153,5 @@
                     filename="libgazebo_ros_diff_drive.so">
                 <rosDebugLevel>Debug</rosDebugLevel>
-                <publishWheelTF>true</publishWheelTF>
+                <publishWheelTF>false</publishWheelTF>
                 <robotNamespace>/</robotNamespace>
                 <publishTf>1</publishTf>

File: mbot_description/urdf/xacro/gazebo/mbot_camera.xacro (robot description, xacro)
@@ -13,4 +13,4 @@
     </joint>
     <xacro:usb_camera prefix="camera"/>
-    <xacro:mbot_base_gazebo/>
+    <!-- <xacro:mbot_base_gazebo/> -->
 </robot>

File: mbot_description/urdf/xacro/gazebo/mbot_kinect.xacro (robot description, xacro)
@@ -13,4 +13,4 @@
     </joint>
     <xacro:kinect_camera prefix="kinect"/>
-    <xacro:mbot_base_gazebo/>
+    <!-- <xacro:mbot_base_gazebo/> -->
 </robot>

File: mbot_description/urdf/xacro/gazebo/mbot_laser.xacro (robot description, xacro)
@@ -3,5 +3,5 @@
     <xacro:include filename="$(find mbot_description)/urdf/xacro/gazebo/mbot_base.xacro" />
     <xacro:include filename="$(find mbot_description)/urdf/xacro/sensors/lidar_gazebo.xacro" />
-    <xacro:property name="lidar_offset_x" value="0" />
+    <xacro:property name="lidar_offset_x" value="0.1" />
     <xacro:property name="lidar_offset_y" value="0" />
     <xacro:property name="lidar_offset_z" value="0.105" />
